File: SmartDimmer.kicad_pcb (KiCad board)
At the start: 4 copper layers, 40 x 75 mm, 86 parts, among them J1 Conn_01x02, J10 Conn_01x02, J11 Conn_01x02, J12 Conn_01x02, J13 Conn_01x02, J2 Conn_01x02, J3 Conn_01x04, J4 Conn_01x02, J5 Conn_01x02, J6 Conn_01x05, J7 Conn_01x08, J8 Conn_01x02, J9 Conn_01x08, Q1 2N7000, Q2 2N7000, Q3 2N7000, Q4 2N7000, Q5 Q_NPN_EBC, Q6 Q_NPN_EBC, SW1 SW_Push, T1 Conn_01x01, T2 Conn_01x01, U1 AT42QT1010-TSHR, U10 ACS712, U11 ACS712, U2 ESP32-WROOM, U3 AT42QT1010-TSHR, U4 FL5160, U5 FL5160, U6 IPD50R399CP, U7 IPD50R399CP, U8 IPD50R399CP, U9 IPD50R399CP

Commit message: NewLayout
Parts:
- removed Q5, Q6: Q_NPN_EBC, Package_TO_SOT_SMD:SOT-23_Handsoldering
- added C21: 1nF, Capacitor_SMD:C_1206_3216Metric_Pad1.42x1.75mm_HandSolder, F.Cu at (134.5, 145.0)
- added C22: 1nF, Capacitor_SMD:C_1206_3216Metric_Pad1.42x1.75mm_HandSolder, F.Cu at (134.5, 147.5)
- added R31: 35K, Resistor_SMD:R_1206_3216Metric_Pad1.42x1.75mm_HandSolder, F.Cu at (142.5, 175.0)
- added RX1: 2K2, Resistor_SMD:R_1206_3216Metric_Pad1.42x1.75mm_HandSolder, F.Cu at (142.5, 177.5)
- added U12: IPD50R399CP, Package_TO_SOT_SMD:TO-252-2, B.Cu at (98.5, 132.9)
- added U13: IPD50R399CP, Package_TO_SOT_SMD:TO-252-2, B.Cu at (91.0, 132.6)
- added U14: IPD50R399CP, Package_TO_SOT_SMD:TO-252-2, B.Cu at (113.5, 132.9)
- added U15: IPD50R399CP, Package_TO_SOT_SMD:TO-252-2, B.Cu at (106.0, 132.6)
- added U16: ACS712, Package_SO:SOIC-8_3.9x4.9mm_P1.27mm, F.Cu at (99.9, 134.5)
- added U17: ACS712, Package_SO:SOIC-8_3.9x4.9mm_P1.27mm, F.Cu at (111.4, 134.5)
- C1, C4: value 100nF -> 3uF; moved to F.Cu
- C10, C12, C9, D1, D2, D3, J1, J2, J4, Q1, Q2, R1: moved to F.Cu
- C11, C8: value 3uF -> 100nF; moved to F.Cu
- C13: value 2nF -> 4.7nF; moved to F.Cu
- C14: value 2nF -> 5pF; moved to F.Cu
- C15, C16: value 22nF -> 2nF; moved to F.Cu
- C17, C18: value 100nF -> 22nF; moved to F.Cu
- C19, C20: value 1nF -> 100nF; moved to F.Cu
- C2, C5: value 4.7nF -> 100nF; moved to F.Cu
- C3: value 5pF -> 3uF; moved to F.Cu
- C6: value 5pF -> 4.7nF; moved to F.Cu
- C7: value 100nF -> 5pF; moved to F.Cu
- J3: value Conn_01x04 -> Conn_01x02; footprint Connector_PinHeader_2.54mm:PinHeader_1x04_P2.54mm_Vertical -> Connector_PinHeader_2.54mm:PinHeader_1x02_P2.54mm_Vertical; moved to F.Cu
- J5: value Conn_01x02 -> Conn_01x08; footprint Connector_PinHeader_2.54mm:PinHeader_1x02_P2.54mm_Vertical -> Connector_PinHeader_2.54mm:PinHeader_1x08_P2.54mm_Vertical; moved to F.Cu
- J6: value Conn_01x05 -> Conn_01x04; footprint Connector_PinHeader_2.54mm:PinHeader_1x05_P2.54mm_Vertical -> Connector_PinHeader_2.54mm:PinHeader_1x04_P2.54mm_Vertical; moved to F.Cu
- J8: value Conn_01x02 -> Conn_01x05; footprint Connector_PinHeader_2.54mm:PinHeader_1x02_P2.54mm_Vertical -> Connector_PinHeader_2.54mm:PinHeader_1x05_P2.54mm_Vertical; moved to F.Cu
- J9: value Conn_01x08 -> Conn_01x02; footprint Connector_PinHeader_2.54mm:PinHeader_1x08_P2.54mm_Vertical -> Connector_PinHeader_2.54mm:PinHeader_1x02_P2.54mm_Vertical
- Q3, Q4: value 2N7000 -> Q_NPN_EBC; moved to F.Cu
- R10, R9: value 10k -> 10K
- R11, R12: value 100k -> 10K
- R15, R16: value 82M -> 10k
- R17: value 2M -> 100K; moved to F.Cu
- R18: value 1K -> 82M; moved to F.Cu
- R19: value 2M -> 82M
- R2: value 10k -> 2K2; moved to F.Cu
- R20: value 2M -> 100K
- R21: value 1K -> 2M; moved to F.Cu
- R22: value 2M -> 1K
- R23: value 350K -> 2M
- R24, R26: value 35K -> 2M
- R25: value 350K -> 1K
- R27: value 1K2 -> 68R
- R28: value 1K2 -> 350K
- R29: value 2K2 -> 35K
- R3, R4, R6: value 10k -> 10K; moved to F.Cu
- R30: value 2K2 -> 350K
- R5: value 100K -> 10K; moved to F.Cu
- R7: value 68R -> 100R; moved to F.Cu
- R8: value 100K -> 100R; moved to F.Cu
- SW1: footprint Button_Switch_SMD:SW_SPST_FSMSM -> Button_Switch_SMD:SW_SPST_PTS645; moved to F.Cu
- U1: value AT42QT1010-TSHR -> ESP32-WROOM; footprint Package_TO_SOT_SMD:SOT-23-6 -> ESP32-footprints-Lib:ESP32-WROOM; moved to F.Cu
- U10, U11: value ACS712 -> FL5160; footprint Package_SO:SOIC-8_3.9x4.9mm_P1.27mm -> Package_SO:SSOP-10_3.9x4.9mm_P1.00mm; moved to F.Cu
- U2: value ESP32-WROOM -> TCMT1100; footprint ESP32-footprints-Lib:ESP32-WROOM -> Package_SO:SOP-4_4.4x2.8mm_P1.27mm; moved to F.Cu
- U3: value AT42QT1010-TSHR -> TCMT1100; footprint Package_TO_SOT_SMD:SOT-23-6 -> Package_SO:SOP-4_4.4x2.8mm_P1.27mm; moved to F.Cu
- U4, U5: value FL5160 -> TCMT1100; footprint Package_SO:SSOP-10_3.9x4.9mm_P1.00mm -> Package_SO:SOP-4_4.4x2.8mm_P1.27mm; moved to F.Cu
- U6, U7: value IPD50R399CP -> TCMT1100; footprint Package_TO_SOT_SMD:TO-252-2 -> Package_SO:SOP-4_4.4x2.8mm_P1.27mm
- U8, U9: value IPD50R399CP -> AT42QT1010-TSHR; footprint Package_TO_SOT_SMD:TO-252-2 -> Package_TO_SOT_SMD:SOT-23-6
- moved R29 73.4 mm to (142.5, 170.0), turned to 0 degrees
- moved R30 70.7 mm to (142.5, 172.5), turned to 0 degrees
- moved R28 69.8 mm to (142.5, 167.5), turned to 0 degrees
- moved R24 67.4 mm to (142.5, 157.5)
- moved R23 64.5 mm to (142.5, 155.0)
- moved R2 64.2 mm to (142.5, 102.5), turned to 0 degrees
- moved R27 62.9 mm to (142.5, 165.0), turned to 0 degrees
- moved R1 60.8 mm to (142.5, 100.0), turned to 0 degrees
- moved R4 59.9 mm to (142.5, 107.5)
- moved R6 59.2 mm to (142.5, 112.5)
- moved R5 59.2 mm to (142.5, 110.0), turned to 0 degrees
- moved R3 58.5 mm to (142.5, 105.0)
- moved R10 56.7 mm to (142.5, 122.5), turned to 0 degrees
- moved R19 53.9 mm to (142.5, 145.0), turned to 0 degrees
- moved R22 52.2 mm to (142.5, 152.5), turned to 0 degrees
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Connections:
- C12 pad 1: Net-(C12-Pad1) -> GND_PWR
- C12 pad 2: GND_PWR -> Net-(C12-Pad2)
- C13 pad 1: /PWR_1 -> Net-(C13-Pad1)
- C14 pad 1: /PWR_6 -> Net-(C14-Pad1)
- C14 pad 2: Net-(C14-Pad2) -> GND
- C15 pad 1: GND_PWR -> /PWR_1
- C16 pad 1: GND_PWR -> /PWR_6
- C19 pad 1: Net-(C19-Pad1) -> GND_PWR
- C19 pad 2: GND_PWR -> Net-(C19-Pad2)
- C2 pad 1: Net-(C2-Pad1) -> VCC
- C2 pad 2: Net-(C2-Pad2) -> GND
- C20 pad 1: Net-(C20-Pad1) -> GND_PWR
- C20 pad 2: GND_PWR -> Net-(C11-Pad1)
- C3 pad 2: GND -> Net-(C3-Pad2)
- C4 pad 1: VCC -> Net-(C4-Pad1)
- C4 pad 2: GND -> Net-(C3-Pad2)
- C5 pad 1: Net-(C5-Pad1) -> VCC
- C5 pad 2: Net-(C5-Pad2) -> GND
- C6 pad 2: GND -> Net-(C6-Pad2)
- C7 pad 1: Net-(C17-Pad2) -> Net-(C7-Pad1)
- C7 pad 2: GND_PWR -> GND
- C8 pad 1: GND_PWR -> VCC
- C8 pad 2: Net-(C8-Pad2) -> GND
- C9 pad 1: Net-(C18-Pad2) -> Net-(C19-Pad2)
- J2 pad 1: VCC -> Net-(J2-Pad1)
- J2 pad 2: Net-(J2-Pad2) -> GND
- J3 pad 1: Net-(J2-Pad2) -> Net-(J3-Pad1)
- J4 pad 1: Net-(J4-Pad1) -> VCC
- J4 pad 2: GND -> Net-(J4-Pad2)
- J5 pad 2: Net-(J5-Pad2) -> Net-(C3-Pad1)
- J6 pad 1: GND -> Net-(J4-Pad2)
- J6 pad 2: VCC -> Net-(J6-Pad2)
- J6 pad 3: Gain -> Net-(J6-Pad3)
- J6 pad 4: Out -> GND
- J7 pad 1: VCC -> (no net)
- J7 pad 2: DIM_Control_1 -> Net-(J7-Pad2)
- J7 pad 3: DIM_MODE_1 -> Net-(J7-Pad3)
- J7 pad 4: Current_Meas_1 -> Net-(J7-Pad4)
- J7 pad 5: DIM_Control_2 -> Net-(J7-Pad5)
- J7 pad 6: DIM_MODE_2 -> Net-(J7-Pad6)
- J7 pad 7: Current_Meas_2 -> Net-(J7-Pad7)
- J7 pad 8: GND -> GND_PWR
- J8 pad 1: VCC -> GND
- J8 pad 2: GND -> VCC
- J9 pad 1: VCC_PWR -> VCC
- J9 pad 2: Net-(J9-Pad2) -> GND
- Q1 pad 3: Net-(J3-Pad2) -> Net-(J6-Pad2)
- Q2 pad 3: Net-(J3-Pad3) -> Net-(J6-Pad3)
- Q3 pad 1: Net-(J9-Pad3) -> Net-(C10-Pad2)
- Q3 pad 2: VCC_PWR -> /HV_6
- Q3 pad 3: Net-(Q3-Pad3) -> /HV_8
- Q4 pad 1: Net-(J9-Pad6) -> Net-(C12-Pad2)
- Q4 pad 2: VCC_PWR -> /HV_9
- Q4 pad 3: Net-(Q4-Pad3) -> /HV_5
- R1 pad 2: TX_3V3 -> Net-(J2-Pad1)
- R10 pad 1: VCC_PWR -> Net-(J5-Pad6)
- R10 pad 2: Net-(J9-Pad6) -> Net-(C3-Pad2)
- R11 pad 1: Net-(C11-Pad1) -> Net-(J5-Pad4)
- R11 pad 2: Net-(J9-Pad2) -> Net-(R11-Pad2)
- R12 pad 1: Net-(C12-Pad1) -> Net-(J5-Pad7)
- R12 pad 2: Net-(J9-Pad5) -> Net-(R12-Pad2)
- R13 pad 1: Net-(C17-Pad2) -> VCC
- R13 pad 2: Net-(Q3-Pad3) -> TX_3V3
- R14 pad 1: Net-(C18-Pad2) -> VCC
- R14 pad 2: Net-(Q4-Pad3) -> RX_3V3
- R15 pad 1: Net-(C13-Pad2) -> Net-(J4-Pad2)
- R15 pad 2: Net-(C18-Pad2) -> Net-(J6-Pad2)
- R16 pad 1: Net-(C17-Pad2) -> Net-(J4-Pad2)
- R16 pad 2: Net-(C14-Pad2) -> Net-(J6-Pad3)
- R17 pad 1: /PWR_6 -> Net-(C7-Pad1)
- R17 pad 2: Net-(R17-Pad2) -> Net-(C6-Pad1)
- R18 pad 2: Net-(R18-Pad2) -> Net-(C11-Pad1)
- R19 pad 1: /PWR_4 -> Net-(C19-Pad2)
- R19 pad 2: Net-(R19-Pad2) -> Net-(C16-Pad2)
- R2 pad 1: VCC -> Net-(R2-Pad1)
- R2 pad 2: RX_3V3 -> DIM_Control_1
- R20 pad 1: /PWR_1 -> Net-(C14-Pad1)
- R20 pad 2: Net-(R20-Pad2) -> Net-(C13-Pad1)
- R21 pad 1: Net-(C16-Pad2) -> /PWR_6
- R22 pad 1: /PWR_2 -> Net-(C17-Pad2)
- R23 pad 1: 230VAC -> /PWR_4
- R23 pad 2: /HV_6 -> Net-(R23-Pad2)
- R24 pad 1: 230VAC -> /PWR_1
- R24 pad 2: /HV_8 -> Net-(R24-Pad2)
- R25 pad 1: 230VAC -> Net-(C18-Pad2)
- R25 pad 2: /HV_9 -> Net-(R25-Pad2)
- R26 pad 1: 230VAC -> /PWR_2
- R26 pad 2: /HV_5 -> Net-(R26-Pad2)
- R27 pad 1: Net-(R27-Pad1) -> Net-(D1-Pad1)
- R27 pad 2: Net-(J9-Pad4) -> GND
- R28 pad 1: Net-(R28-Pad1) -> 230VAC
- R28 pad 2: Net-(J9-Pad7) -> /HV_6
- R29 pad 1: GND_PWR -> 230VAC
- R29 pad 2: Net-(J9-Pad4) -> /HV_8
- R3 pad 1: Net-(J2-Pad2) -> Net-(R3-Pad1)
- R3 pad 2: Net-(J3-Pad2) -> Current_Meas_2
- R30 pad 1: GND_PWR -> 230VAC
- R30 pad 2: Net-(J9-Pad7) -> /HV_9
- R4 pad 1: Net-(J2-Pad2) -> Net-(R3-Pad1)
- R4 pad 2: Net-(J3-Pad3) -> Current_Meas_1
- R5 pad 2: Net-(C2-Pad1) -> Net-(C3-Pad2)
- R6 pad 1: VCC -> Net-(C3-Pad2)
- R6 pad 2: Net-(J4-Pad1) -> Net-(C4-Pad1)
- R7 pad 1: Net-(D1-Pad1) -> Net-(R7-Pad1)
- R8 pad 1: Net-(C6-Pad1) -> Net-(R8-Pad1)
- R8 pad 2: Net-(C5-Pad1) -> GND
- R9 pad 1: VCC_PWR -> Net-(J5-Pad3)
- R9 pad 2: Net-(J9-Pad3) -> Net-(C3-Pad2)
- T1 pad 1: Net-(C6-Pad1) -> Net-(C7-Pad1)
- T2 pad 1: Net-(C3-Pad1) -> Net-(C14-Pad1)
- U1 pad 1: TOUCH_2 -> GND
- U1 pad 2: GND -> VCC
- U1 pad 3: Net-(C2-Pad1) -> VCC
- U1 pad 4: Net-(C2-Pad2) -> (no net)
- U1 pad 5: VCC -> (no net)
- U1 pad 6: TOUCH_SYNC -> (no net)
- U10 pad 1: /PWR_5 -> Net-(C16-Pad2)
- U10 pad 2: /PWR_5 -> Net-(J7-Pad2)
- U10 pad 3: /PWR_4 -> Net-(C19-Pad2)
- U10 pad 4: /PWR_4 -> Net-(J7-Pad3)
- U10 pad 6: Net-(C19-Pad1) -> Net-(C10-Pad2)
- U10 pad 7: Net-(R27-Pad1) -> /HV_6
- U10 pad 8: Net-(C17-Pad2) -> Net-(R23-Pad2)
- U11 pad 1: /PWR_3 -> Net-(C15-Pad2)
- U11 pad 2: /PWR_3 -> Net-(J7-Pad5)
- U11 pad 3: /PWR_2 -> Net-(C11-Pad1)
- U11 pad 4: /PWR_2 -> Net-(J7-Pad6)
- U11 pad 6: Net-(C20-Pad1) -> Net-(C12-Pad2)
- U11 pad 7: Net-(R28-Pad1) -> /HV_9
- U11 pad 8: Net-(C18-Pad2) -> Net-(R26-Pad2)
- U2 pad 1: GND -> Net-(R2-Pad1)
- U2 pad 2: VCC -> GND
- U2 pad 3: VCC -> Net-(C3-Pad1)
- U2 pad 4: Net-(U2-Pad4) -> Net-(J5-Pad1)
- U3 pad 1: TOUCH_1 -> Net-(RX1-Pad1)
- U3 pad 3: Net-(C5-Pad1) -> Net-(C4-Pad1)
- U3 pad 4: Net-(C5-Pad2) -> Net-(J5-Pad1)
- U4 pad 1: Net-(C14-Pad2) -> Net-(R11-Pad2)
- U4 pad 2: Net-(C11-Pad1) -> Net-(C3-Pad2)
- U4 pad 3: Net-(C17-Pad2) -> GND
- U4 pad 4: Net-(Q3-Pad3) -> Current_Meas_1
- U5 pad 1: Net-(C13-Pad2) -> Net-(R12-Pad2)
- U5 pad 2: Net-(C12-Pad1) -> Net-(C3-Pad2)
- U5 pad 3: Net-(C18-Pad2) -> GND
- U5 pad 4: Net-(Q4-Pad3) -> Current_Meas_2
- U6 pad 1: Net-(C15-Pad2) -> DIM_MODE_1
- U6 pad 2: /PWR_6 -> Net-(R7-Pad1)
- U6 pad 3: GND_PWR -> Net-(J5-Pad3)
- U7 pad 1: Net-(C15-Pad2) -> DIM_MODE_2
- U7 pad 2: /PWR_4 -> Net-(R8-Pad1)
- U7 pad 3: GND_PWR -> Net-(J5-Pad6)
- U8 pad 1: Net-(C16-Pad2) -> TOUCH_2
- U8 pad 2: /PWR_1 -> GND
- U8 pad 3: GND_PWR -> Net-(C6-Pad1)
- U9 pad 1: Net-(C16-Pad2) -> TOUCH_1
- U9 pad 2: /PWR_2 -> GND
- U9 pad 3: GND_PWR -> Net-(C13-Pad1)
Other:
- board text removed: "+ -"
- board text removed: "GND RX TX SIG_REF"
- board text removed: "GND VDD GAIN OUT A/R"
- board text removed: "IO14 IO12"
- board text removed: "IO5 IO4"
- board text removed: "RUN /PRG"
- board text removed: "Reset"
- board text removed: "Short if SIG_REF = 3V3"
- board text removed: "SmartDimmer V2.0"

Commit message: RoutingDone
Parts:
- removed RX1: 2K2, Resistor_SMD:R_1206_3216Metric_Pad1.42x1.75mm_HandSolder
- added R32: 2K2, Resistor_SMD:R_1206_3216Metric_Pad1.42x1.75mm_HandSolder, B.Cu at (111.0, 95.0)
- C13, C14, C3, C4, C5, C6, C7, C8, J11, J12, J13, R10, R11, R12, R17, R2, R20, R3, R4, R5, R6, R7, R8, R9, U2, U3, U4, U5, U6, U7, U8, U9: moved to B.Cu
- moved R27 96.8 mm to (88.0, 85.0), turned to 90 degrees
- moved R17 77.0 mm to (93.0, 81.0), turned to 270 degrees
- moved R20 74.0 mm to (93.0, 92.5), turned to 270 degrees
- moved R28 66.8 mm to (87.2, 130.0), turned to 90 degrees
- moved R29 66.2 mm to (89.8, 130.0), turned to 90 degrees
- moved R30 65.6 mm to (92.5, 130.0), turned to 90 degrees
- moved R31 65.6 mm to (94.8, 130.0), turned to 90 degrees
- moved R16 65.6 mm to (115.0, 78.0), turned to 270 degrees
- moved R15 64.6 mm to (112.0, 78.0), turned to 270 degrees
- moved R19 63.3 mm to (84.5, 119.8), turned to 270 degrees
- moved R12 61.6 mm to (102.0, 81.0), turned to 270 degrees
- moved C14 59.3 mm to (89.0, 89.5), turned to 180 degrees
- moved C7 58.6 mm to (89.0, 78.0), turned to 180 degrees
- moved R8 58.3 mm to (97.0, 81.0), turned to 90 degrees
- moved R11 58.1 mm to (104.5, 81.0), turned to 270 degrees
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Connections:
- R18 pad 2: Net-(C11-Pad1) -> GND_PWR
- R19 pad 1: Net-(C19-Pad2) -> Net-(C16-Pad2)
- R19 pad 2: Net-(C16-Pad2) -> GND_PWR
Routing:
- net GND: track 0.00 -> 189.3 mm, vias 0 -> 9
- net GND_PWR: track 0.00 -> 117.1 mm, vias 0 -> 9
- net VCC: track 0.00 -> 106.2 mm, vias 0 -> 6
- net Net-(SW1-Pad1): track 0.00 -> 70.8 mm, vias 0 -> 4
- net Net-(C7-Pad1): track 0.00 -> 67.0 mm, vias 0 -> 1
- net Net-(R21-Pad2): track 0.00 -> 63.1 mm, vias 0 -> 4
- net Net-(C4-Pad1): track 0.00 -> 55.2 mm, vias 0 -> 1
- net Net-(C3-Pad2): track 0.00 -> 54.7 mm, vias 0 -> 3
- net Net-(C3-Pad1): track 0.00 -> 52.5 mm, vias 0 -> 1
- net /HV_9: track 0.00 -> 50.1 mm, vias 0 -> 6
- net /PWR_1: track 0.00 -> 46.7 mm, vias 0 -> 6
- net Net-(C15-Pad2): track 0.00 -> 44.2 mm, vias 0 -> 2
- net Net-(J5-Pad1): track 0.00 -> 43.4 mm, vias 0 -> 3
- net TOUCH_SYNC: track 0.00 -> 41.9 mm, vias 0 -> 1
- net Net-(J5-Pad4): track 0.00 -> 41.7 mm, vias 0 -> 4
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Other:
- copper layers 4 -> 2
