File: SmartDimmer.kicad_pcb (KiCad board)
At the start: 2 copper layers, 40 x 75 mm, 94 parts, among them J1 Conn_01x02, J10 Conn_01x02, J11 Conn_01x02, J12 Conn_01x02, J13 Conn_01x02, J2 Conn_01x02, J3 Conn_01x02, J4 Conn_01x02, J5 Conn_01x08, J6 Conn_01x04, J7 Conn_01x08, J8 Conn_01x05, J9 Conn_01x02, Q1 2N7000, Q2 2N7000, Q3 Q_NPN_EBC, Q4 Q_NPN_EBC, SW1 SW_Push, T1 Conn_01x01, T2 Conn_01x01, U1 ESP32-WROOM, U10 FL5160, U11 FL5160, U12 IPD50R399CP, U13 IPD50R399CP, U14 IPD50R399CP, U15 IPD50R399CP, U16 ACS712, U17 ACS712, U2 TCMT1100, U3 TCMT1100, U4 TCMT1100, U5 TCMT1100, U6 TCMT1100, U7 TCMT1100, U8 AT42QT1010-TSHR, U9 AT42QT1010-TSHR

Commit message: aestetic change
Other:
- board text added: "230VAC"
- board text added: "DIM1"
- board text added: "DIM2"
Changed lines of the file:
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@@
   (general
     (thickness 1.6)
-    (drawings 17)
+    (drawings 20)
     (tracks 1355)
     (zones 0)
@@
     (34 B.Paste user hide)
     (35 F.Paste user hide)
-    (36 B.SilkS user hide)
+    (36 B.SilkS user)
     (37 F.SilkS user)
-    (38 B.Mask user hide)
+    (38 B.Mask user)
     (39 F.Mask user)
     (40 Dwgs.User user)
@@
     (tags "resistor handsolder")
     (attr smd)
-    (fp_text reference R1 (at 0 -2) (layer F.SilkS)
+    (fp_text reference R1 (at -0.0125 1.7) (layer F.SilkS)
       (effects (font (size 1 1) (thickness 0.15)))
     )
@@
     (descr "Through hole straight pin header, 1x01, 2.54mm pitch, single row")
     (tags "Through hole pin header THT 1x01 2.54mm single row")
-    (fp_text reference T2 (at 3 0 180) (layer F.SilkS)
+    (fp_text reference T2 (at 2.1 0.2 180) (layer F.SilkS)
       (effects (font (size 1 1) (thickness 0.15)))
     )
@@
     )
   )
+  (gr_text DIM2 (at 111.4 140.1) (layer F.SilkS)
+    (effects (font (size 1.5 1.5) (thickness 0.3)))
+  )
+  (gr_text DIM1 (at 100 140.2) (layer F.SilkS)
+    (effects (font (size 1.5 1.5) (thickness 0.3)))
+  )
+  (gr_text 230VAC (at 88.2 140.3) (layer F.SilkS)
+    (effects (font (size 1.5 1.5) (thickness 0.3)))
+  )
   (target plus (at 80 110) (size 5) (width 0.15) (layer Edge.Cuts))
